Commit message: Attached end effector to ur5 arm

File: robots/ur5_barrett.urdf.xacro (robot description, xacro)
@@ -1,30 +1,13 @@
 <?xml version="1.0"?>
-<robot name="bhand" xmlns:xacro="http://ros.org/wiki/xacro">
-	<!-- Available choices: bh282.urdf.xacro, bh280.urdf.xacro -->
+<robot name="ur5_barrett" xmlns:xacro="http://ros.org/wiki/xacro">
+	<!-- barrett hand -->
 	<xacro:include filename="$(find barrett_hand_description)/urdf/bh280.urdf.xacro" />
-	<!-- z-coordinate is not 0 because otherwise the hand base tilts when the simulation is started -->
-	<link name="base_link">
-		<visual>
-		  <origin xyz="0 0 0.01" rpy="0 0 0" />
-		  <geometry>
-			 <box size="0.001 0.001 0.001" />
-		  </geometry>
-		</visual>
-		<collision>
-		  <origin xyz="0 0 0.01" rpy="0 0 0" />
-		  <geometry>
-			<box size="0.001 0.001 0.001" />
-		  </geometry>
-		</collision>
-	</link>
-	<joint name="hand_joint" type="fixed">
-		 <origin xyz="0 0 0" rpy="0 0 0" />
-		 <parent link="base_link"/>
-		 <child link="hand_base_link"/>
-	</joint>
-	<link name="hand_base_link"/>
-	<xacro:bhand_macro name="bh" parent="hand_base_link">
-		<origin xyz="0 0 0" rpy="0 0 0" />
-	</xacro:bhand_macro>
+	<!-- ur5 -->
+  <xacro:include filename="$(find ur_description)/urdf/ur5.urdf.xacro" />
+	<!-- fixing barrett hand to the ur5 -->
+	<xacro:bhand_macro parent="ee_link" name="bh">
+  		<origin xyz="0 0 0" rpy="1.57 0 1.57" />
+  	</xacro:bhand_macro>
+	<!-- Hand attached to the arm -->
 	<gazebo>
 	    <plugin name="ros_control" filename="libgazebo_ros_control.so">
@@ -34,12 +17,4 @@
 	    </plugin>
     </gazebo>
-</robot>
-<?xml version="1.0"?>
-<robot xmlns:xacro="http://ros.org/wiki/xacro"
-       name="ur5" >
-  <!-- common stuff -->
-  <xacro:include filename="$(find ur_description)/urdf/common.gazebo.xacro" />
-  <!-- ur5 -->
-  <xacro:include filename="$(find ur_description)/urdf/ur5.urdf.xacro" />
   <!-- arm -->
   <xacro:ur5_robot prefix="" joint_limited="false"/>
